File: hardware/v6.brd (EAGLE design)
At the start: 40.1 x 88.1 mm, 50 parts, among them IC1 VCNL3040, IC2 SN74AUP1T58DRYR, IC3 SN74AUP1T58DCKR, IC4 SN74AUP1T58DCKR, IC7 SN74AUP1T58DRYR, J3 62701021621, U1 UG-2864HSWEG01

Commit message: First commit
Connections:
- removed net 3V3: C3.2, C4.2, R4.2, R6.2, R7.2, U1.11, U1.6, U1.9
- net +3V3: now also C3.2, C4.2, R4.2, R6.2, R7.2, U1.11, U1.6, U1.9
Routing:
- net +3V3: track 172.0 -> 198.4 mm, vias 7 -> 12
- net 3V3: track 20.5 -> 0.00 mm, vias 4 -> 0
- added copper zone on layer 16, net +3V3
- removed copper zone on layer 16, net 3V3
Changed lines of the file:
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@@
 <wire x1="33.25" y1="61.375" x2="33.275" y2="61.35" width="0.254" layer="1"/>
-</signal>
-<signal name="3V3">
-<contactref element="U1" pad="11"/>
-<contactref element="U1" pad="6"/>
-<contactref element="U1" pad="9"/>
-<contactref element="C3" pad="2"/>
-<contactref element="C4" pad="2"/>
-<contactref element="R4" pad="2"/>
-<contactref element="R7" pad="2"/>
-<contactref element="R6" pad="2"/>
-<wire x1="24.36" y1="8.518" x2="24.36" y2="10.44" width="0.4064" layer="16"/>
-<polygon width="0.1524" layer="16">
-<vertex x="19.45" y="20.95"/>
-<vertex x="19.45" y="16.95"/>
-<vertex x="21.45" y="17"/>
-<vertex x="23.2" y="18.75"/>
-<vertex x="23.2" y="21.4"/>
-<vertex x="19.5" y="21.4"/>
-</polygon>
-<wire x1="26.212" y1="22.806" x2="26.212" y2="21.938" width="0.3048" layer="16"/>
-<wire x1="26.212" y1="21.938" x2="26.2" y2="21.95" width="0.3048" layer="16"/>
-<via x="26.2" y="21.95" extent="1-16" drill="0.3" shape="octagon"/>
-<wire x1="26.2" y1="21.95" x2="22.45" y2="21.95" width="0.3048" layer="1"/>
-<wire x1="22.45" y1="21.95" x2="21.3" y2="20.8" width="0.3048" layer="1"/>
-<via x="21.3" y="20.8" extent="1-16" drill="0.3" shape="octagon"/>
-<wire x1="21.3" y1="20.8" x2="22.645" y2="20.9" width="0.3048" layer="16"/>
-<wire x1="22.645" y1="20.9" x2="22.66" y2="20.885" width="0.3048" layer="16"/>
-<wire x1="24.36" y1="10.44" x2="24.36" y2="11.41" width="0.3048" layer="16"/>
-<wire x1="24.36" y1="11.41" x2="24.4" y2="11.45" width="0.3048" layer="16"/>
-<via x="24.4" y="11.45" extent="1-16" drill="0.3" shape="octagon"/>
-<wire x1="24.4" y1="11.45" x2="24.4" y2="14.85" width="0.3048" layer="1"/>
-<wire x1="24.4" y1="14.85" x2="21.3" y2="17.95" width="0.3048" layer="1"/>
-<via x="21.3" y="17.95" extent="1-16" drill="0.3" shape="octagon"/>
-<wire x1="21.3" y1="17.95" x2="21.3" y2="18.6" width="0.3048" layer="16"/>
-<wire x1="21.3" y1="18.6" x2="21.65" y2="18.95" width="0.3048" layer="16"/>
-<wire x1="21.65" y1="18.95" x2="22.642" y2="18.95" width="0.3048" layer="16"/>
-<wire x1="22.642" y1="18.95" x2="22.66" y2="18.932" width="0.3048" layer="16"/>
 </signal>
 <signal name="GPIO10_MOSI">
@@
 <via x="29.95" y="20.875" extent="1-16" drill="0.3" shape="octagon"/>
 <wire x1="29.95" y1="20.875" x2="29.575" y2="21.25" width="0.254" layer="1"/>
-<wire x1="29.575" y1="21.25" x2="29.575" y2="27" width="0.254" layer="1"/>
+<wire x1="29.575" y1="21.25" x2="29.575" y2="22.15" width="0.254" layer="1"/>
+<wire x1="29.575" y1="22.15" x2="29.85" y2="22.425" width="0.254" layer="1"/>
+<wire x1="29.575" y1="22.7" x2="29.575" y2="27" width="0.254" layer="1"/>
 <wire x1="29.575" y1="27" x2="30.55" y2="27.975" width="0.254" layer="1"/>
 <wire x1="30.55" y1="27.975" x2="30.55" y2="29.475" width="0.254" layer="1"/>
@@
 <contactref element="R2" pad="2"/>
 <wire x1="32.6" y1="20.885" x2="32.6" y2="22.85" width="0.3048" layer="16"/>
+<contactref element="C4" pad="2"/>
+<contactref element="U1" pad="9"/>
+<contactref element="C3" pad="2"/>
+<contactref element="U1" pad="6"/>
+<contactref element="U1" pad="11"/>
+<contactref element="R4" pad="2"/>
+<contactref element="R7" pad="2"/>
+<contactref element="R6" pad="2"/>
+<polygon width="0.1524" layer="16">
+<vertex x="19.45" y="20.95"/>
+<vertex x="19.45" y="16.95"/>
+<vertex x="21.45" y="17"/>
+<vertex x="23.2" y="18.75"/>
+<vertex x="23.2" y="21.4"/>
+<vertex x="19.5" y="21.4"/>
+</polygon>
+<wire x1="26.212" y1="22.806" x2="26.212" y2="22.012" width="0.254" layer="16"/>
+<wire x1="26.212" y1="22.012" x2="26.2" y2="22" width="0.254" layer="16"/>
+<via x="26.2" y="22" extent="1-16" drill="0.3" shape="octagon"/>
+<wire x1="26.2" y1="22" x2="22.5" y2="22" width="0.254" layer="1"/>
+<wire x1="22.5" y1="22" x2="21.4" y2="20.9" width="0.254" layer="1"/>
+<via x="21.4" y="20.9" extent="1-16" drill="0.3" shape="octagon"/>
+<wire x1="21.4" y1="20.9" x2="22.645" y2="20.9" width="0.254" layer="16"/>
+<wire x1="22.645" y1="20.9" x2="22.66" y2="20.885" width="0.254" layer="16"/>
+<wire x1="24.36" y1="8.518" x2="24.36" y2="10.44" width="0.254" layer="16"/>
+<wire x1="24.36" y1="10.44" x2="24.36" y2="11.69" width="0.254" layer="16"/>
+<wire x1="24.36" y1="11.69" x2="24.35" y2="11.7" width="0.254" layer="16"/>
+<via x="24.35" y="11.7" extent="1-16" drill="0.3" shape="octagon"/>
+<wire x1="24.35" y1="11.7" x2="24.35" y2="15.025" width="0.254" layer="1"/>
+<wire x1="24.35" y1="15.025" x2="21.3" y2="18.075" width="0.254" layer="1"/>
+<via x="21.3" y="18.075" extent="1-16" drill="0.3" shape="octagon"/>
+<wire x1="21.3" y1="18.075" x2="21.3" y2="18.675" width="0.254" layer="16"/>
+<wire x1="21.3" y1="18.675" x2="21.325" y2="18.7" width="0.254" layer="16"/>
+<wire x1="21.325" y1="18.7" x2="21.3" y2="18.7" width="0.254" layer="16"/>
+<wire x1="21.3" y1="18.7" x2="21" y2="19" width="0.254" layer="16"/>
+<wire x1="21" y1="19" x2="21" y2="20.5" width="0.254" layer="16"/>
+<wire x1="21" y1="20.5" x2="21.4" y2="20.9" width="0.254" layer="16"/>
+<wire x1="26.212" y1="22.806" x2="26.212" y2="23.437" width="0.254" layer="16"/>
+<wire x1="26.212" y1="23.437" x2="26.45" y2="23.675" width="0.254" layer="16"/>
+<wire x1="26.45" y1="23.675" x2="28.5" y2="23.675" width="0.254" layer="16"/>
+<wire x1="29.575" y1="22.7" x2="29.85" y2="22.425" width="0.254" layer="1"/>
+<via x="29.85" y="22.425" extent="1-16" drill="0.3" shape="octagon"/>
+<wire x1="29.85" y1="22.425" x2="29.75" y2="22.425" width="0.254" layer="16"/>
+<wire x1="29.75" y1="22.425" x2="28.5" y2="23.675" width="0.254" layer="16"/>
 </signal>
 <signal name="INT">

Commit message: Changed connector
Parts:
- removed J3: 62701021621, Eagle_WR-BHD (rev22c):62701021621
- added J8: 62501021621, Eagle_WR-BHD (rev22c):62501021621
- added Q3: (no value), adafruit:SOT23
- added R8, R9: 10k, rcl:R0603
Connections:
- removed net N$17: JP5.1, JP8.1, LED1.4-DIN
- new net LED_IN: JP8.1, LED1.4-DIN, Q3.3, R9.1
- new net N$2: JP5.1, Q3.2, R8.1
- net +3V3: now also Q3.1, R8.2
- net +5V: now also J8.1, R9.2; no longer J3.1
- net 10MHZ_RPI: now also J8.10; no longer J3.10
- net D0: now also J8.2; no longer J3.2
- net D1: now also J8.3; no longer J3.3
- net GND: now also J8.6, J8.8, J8.9; no longer J3.6, J3.8, J3.9
- net PPS_RPI: now also J8.7; no longer J3.7
- net SCL: now also J8.5; no longer J3.5
- net SDA: now also J8.4; no longer J3.4
Routing:
- net N$17: track 29.2 -> 0.00 mm
- net LED_IN: track 0.00 -> 28.0 mm
- net +5V: track 113.5 -> 141.1 mm, vias 3 -> 5
- net +3V3: track 198.4 -> 207.3 mm
- net D0: track 17.2 -> 25.6 mm
- net D1: track 21.3 -> 29.3 mm, vias 2 -> 3
- net SDA: track 154.5 -> 150.0 mm
- net N$2: track 0.00 -> 4.44 mm
- net GND: track 9.56 -> 11.3 mm, vias 94 -> 100
- net 10MHZ_RPI: track 7.93 -> 9.58 mm, vias 0 -> 1
- net SCL: track 150.9 -> 152.0 mm, vias 6 -> 7
- net PPS_RPI: track 6.65 -> 7.77 mm, vias 0 -> 1
