File: hardware/v6.sch (EAGLE design)
At the start: 50 parts, among them IC1 VCNL3040, IC2 SN74AUP1T58DRYR, IC3 SN74AUP1T58DCKR, IC4 SN74AUP1T58DCKR, IC7 SN74AUP1T58DRYR, J3 62701021621, U1 UG-2864HSWEG01

Commit message: First commit
Connections:
- removed net 3V3: C3.2, C4.2, R4.2, R6.2, R7.2, U1.BS1, U1.VBAT, U1.VDD
- net +3V3: now also C3.2, C4.2, R4.2, R6.2, R7.2, U1.BS1, U1.VBAT, U1.VDD
Changed lines of the file:
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@@
-</segment>
-</net>
-<net name="3V3" class="0">
-<segment>
-<wire x1="68.58" y1="88.9" x2="81.28" y2="88.9" width="0.1524" layer="91"/>
-<pinref part="U1" gate="G$1" pin="BS1"/>
-<label x="71.12" y="88.9" size="1.778" layer="95"/>
-</segment>
-<segment>
-<wire x1="81.28" y1="101.6" x2="68.58" y2="101.6" width="0.1524" layer="91"/>
-<pinref part="U1" gate="G$1" pin="VBAT"/>
-<label x="71.12" y="101.6" size="1.778" layer="95"/>
-<pinref part="C3" gate="G$1" pin="2"/>
-</segment>
-<segment>
-<pinref part="U1" gate="G$1" pin="VDD"/>
-<wire x1="81.28" y1="93.98" x2="68.58" y2="93.98" width="0.1524" layer="91"/>
-<label x="71.12" y="93.98" size="1.778" layer="95"/>
-<pinref part="C4" gate="G$1" pin="2"/>
-</segment>
-<segment>
-<wire x1="93.98" y1="147.32" x2="83.82" y2="147.32" width="0.1524" layer="91"/>
-<label x="86.36" y="147.32" size="1.778" layer="95"/>
-<pinref part="R6" gate="G$1" pin="2"/>
-</segment>
-<segment>
-<wire x1="93.98" y1="139.7" x2="83.82" y2="139.7" width="0.1524" layer="91"/>
-<label x="86.36" y="139.7" size="1.778" layer="95"/>
-<pinref part="R7" gate="G$1" pin="2"/>
-</segment>
-<segment>
-<wire x1="27.94" y1="93.98" x2="27.94" y2="96.52" width="0.1524" layer="91"/>
-<wire x1="27.94" y1="96.52" x2="38.1" y2="96.52" width="0.1524" layer="91"/>
-<label x="30.48" y="96.52" size="1.778" layer="95"/>
-<pinref part="R4" gate="G$1" pin="2"/>
 </segment>
 </net>
@@
 </segment>
 </net>
+<net name="+3V3" class="0">
+<segment>
+<pinref part="U1" gate="G$1" pin="VDD"/>
+<wire x1="81.28" y1="93.98" x2="68.58" y2="93.98" width="0.1524" layer="91"/>
+<label x="71.12" y="93.98" size="1.778" layer="95"/>
+<pinref part="C4" gate="G$1" pin="2"/>
+</segment>
+<segment>
+<wire x1="81.28" y1="101.6" x2="68.58" y2="101.6" width="0.1524" layer="91"/>
+<pinref part="U1" gate="G$1" pin="VBAT"/>
+<label x="71.12" y="101.6" size="1.778" layer="95"/>
+<pinref part="C3" gate="G$1" pin="2"/>
+</segment>
+<segment>
+<wire x1="68.58" y1="88.9" x2="81.28" y2="88.9" width="0.1524" layer="91"/>
+<pinref part="U1" gate="G$1" pin="BS1"/>
+<label x="71.12" y="88.9" size="1.778" layer="95"/>
+</segment>
+<segment>
+<wire x1="27.94" y1="93.98" x2="27.94" y2="96.52" width="0.1524" layer="91"/>
+<wire x1="27.94" y1="96.52" x2="38.1" y2="96.52" width="0.1524" layer="91"/>
+<label x="30.48" y="96.52" size="1.778" layer="95"/>
+<pinref part="R4" gate="G$1" pin="2"/>
+</segment>
+<segment>
+<wire x1="93.98" y1="139.7" x2="83.82" y2="139.7" width="0.1524" layer="91"/>
+<label x="86.36" y="139.7" size="1.778" layer="95"/>
+<pinref part="R7" gate="G$1" pin="2"/>
+</segment>
+<segment>
+<wire x1="93.98" y1="147.32" x2="83.82" y2="147.32" width="0.1524" layer="91"/>
+<label x="86.36" y="147.32" size="1.778" layer="95"/>
+<pinref part="R6" gate="G$1" pin="2"/>
+</segment>
+</net>

Commit message: Changed connector
Parts:
- removed J3: 62701021621, Eagle_WR-BHD (rev22c):6270XX21621_62701021621
- added J8: 62501021621, Eagle_WR-BHD (rev22c):6250XX21621_62501021621
- added Q3: (no value), adafruit:MOSFET-NREFLOW
- added R8, R9: 10k, rcl:R-EU_R0603
Connections:
- removed net N$17: JP5.1, JP8.1, LED1.DI
- new net LED_IN: JP8.1, LED1.DI, Q3.D, R9.1
- new net N$2: JP5.1, Q3.S, R8.1
- net +3V3: now also Q3.G, R8.2
- net +5V: now also J8.1, R9.2; no longer J3.1
- net 10MHZ_RPI: now also J8.10; no longer J3.10
- net D0: now also J8.2; no longer J3.2
- net D1: now also J8.3; no longer J3.3
- net GND: now also J8.6, J8.8, J8.9; no longer J3.6, J3.8, J3.9
- net PPS_RPI: now also J8.7; no longer J3.7
- net SCL: now also J8.5; no longer J3.5
- net SDA: now also J8.4; no longer J3.4
Other:
- moved on the sheet: JP5
